File: media_poe_splitter.kicad_sch (KiCad schematic)
At the start: 81 parts, among them IC1 LAN7850-I_8JX, IC2 17791063215, IC3 93AA66C-I/SN, J1 Screw_Terminal_01x02, Q1 DMP3099L-7, X1 7499811120, X2 68710614522, Y1 830055299

Commit message: Fix voltage issues, bigger traces where needed
Signed-off-by: Marc 'risson' Schmitt <marc.schmitt@risson.space>
Parts:
- removed C10, C7: 100nF 25V, 885012206071:885012206071, symbol 885012206071:885012206071
- removed C4: 2.2uF 25V, 885012207079:885012207079, symbol 885012207079:885012207079
- removed C8: 10nF 6.3V, 885012104004:885012104004, symbol 885012104004:885012104004
- removed Q1: DMP3099L-7, DMP3099L-7:DMP3099L-7, symbol DMP3099L-7:DMP3099L-7
- added Q1: SSM3J358R,LF, SSM3J358R,LF:SSM3J358R,LF, symbol SSM3J358R,LF:SSM3J358R_LF
- added R14: 8.2k, RC0603FR-078K2L:RC0603FR-078K2L, symbol RC0603FR-078K2L:RC0603FR-078K2L
- R11, R2: value 330R -> 340R
- R6: value 47.8K -> 48.7K
Connections:
- net GNDA: now also B1.11 (0V2), B1.12 (0V2), C1.2
- net at B1.10 (VOUT2), B1.9 (VOUT2), C1.1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: now also B1.13 (VOUT1), B1.14 (VOUT1), C2.1, Q1.2, R14.1
- net at J2.2, R5.2: now also Q1.1
- net at B1.17 (ADJ): now also R14.2
- net +24V renamed +15V
- net +15V: now also Q1.3
- no-connect marks 33 -> 32
Other:
- note added: "15V -> 3.3V"
- note added: "PoE processing + 15V output"
- note removed: "24V -> 3.3V"
- note removed: "PoE processing + 24V output"
- moved on the sheet: C21, C22, IC2, J1, J2, R5, R6
